File: Stepper_Motor_FOC.kicad_pcb (KiCad board)
At the start: 2 copper layers, 42 x 42 mm, 9 parts, among them J1 Conn_01x04, J2 Conn_01x04, J3 Conn_01x04, J4 Conn_01x04, U1 STM32F103C8Tx, U2 DRV8841, U3 ME3116, U4 MA730, U5 SPX3819M5-L-3-3

Commit message: update sch
Parts:
- added C1: 30PF, Capacitor_SMD:C_0402_1005Metric, F.Cu at (131.1, 119.5)
- added C10: 10uf, Capacitor_SMD:C_0402_1005Metric, F.Cu at (133.9, 114.3)
- added C11: 4.7uF, Capacitor_SMD:C_1206_3216Metric_Pad1.33x1.80mm_HandSolder, F.Cu at (122.7, 111.0)
- added C12: 100nF, Capacitor_SMD:C_0402_1005Metric_Pad0.74x0.62mm_HandSolder, F.Cu at (121.1, 125.0)
- added C13: 100nF, Capacitor_SMD:C_0402_1005Metric_Pad0.74x0.62mm_HandSolder, F.Cu at (132.5, 110.3)
- added C14: 100nF, Capacitor_SMD:C_0402_1005Metric_Pad0.74x0.62mm_HandSolder, F.Cu at (121.3, 117.0)
- added C15: 4.7uF, Capacitor_SMD:C_0402_1005Metric_Pad0.74x0.62mm_HandSolder, F.Cu at (135.8, 110.3)
- added C16: 47uF, Capacitor_SMD:C_1206_3216Metric_Pad1.33x1.80mm_HandSolder, F.Cu at (122.7, 114.3)
- added C17: 100nF, Capacitor_SMD:C_0402_1005Metric_Pad0.74x0.62mm_HandSolder, F.Cu at (127.7, 115.6)
- added C18: 100nF, Capacitor_SMD:C_0402_1005Metric_Pad0.74x0.62mm_HandSolder, F.Cu at (127.7, 117.5)
- added C19: 100nF, Capacitor_SMD:C_0402_1005Metric_Pad0.74x0.62mm_HandSolder, F.Cu at (121.3, 119.0)
- added C2: 4u7, Capacitor_SMD:C_0402_1005Metric, F.Cu at (128.2, 121.5)
- added C20: 4.7uF, Capacitor_SMD:C_0402_1005Metric_Pad0.74x0.62mm_HandSolder, F.Cu at (122.0, 121.0)
- added C21: 47uF, Capacitor_SMD:C_1206_3216Metric_Pad1.33x1.80mm_HandSolder, F.Cu at (111.3, 122.3)
- added C22: 47uF, Capacitor_SMD:C_1206_3216Metric_Pad1.33x1.80mm_HandSolder, F.Cu at (117.3, 122.3)
- added C23: 47uF, Capacitor_SMD:C_1206_3216Metric_Pad1.33x1.80mm_HandSolder, F.Cu at (111.3, 125.7)
- added C3: 100nf, Capacitor_SMD:C_0402_1005Metric, F.Cu at (130.7, 117.5)
- added C4: 30PF, Capacitor_SMD:C_0402_1005Metric, F.Cu at (128.2, 119.5)
- added C5: 100nf, Capacitor_SMD:C_0402_1005Metric, F.Cu at (124.1, 127.0)
- added C6: 100nf, Capacitor_SMD:C_0402_1005Metric, F.Cu at (138.5, 112.3)
- added C7: 100nf, Capacitor_SMD:C_0402_1005Metric, F.Cu at (133.9, 116.2)
- added C8: 100nf, Capacitor_SMD:C_0402_1005Metric, F.Cu at (127.1, 124.9)
- added C9: 100nf, Capacitor_SMD:C_0402_1005Metric, F.Cu at (138.8, 110.3)
- added D1: LED, LED_SMD:LED_0402_1005Metric, F.Cu at (121.2, 127.0)
- added R1: 10K, Resistor_SMD:R_0402_1005Metric, F.Cu at (124.2, 124.9)
- added R2: 1K5, Resistor_SMD:R_0402_1005Metric, F.Cu at (135.6, 112.3)
- added R3: 10K, Resistor_SMD:R_0402_1005Metric, F.Cu at (125.0, 122.9)
- added R4: R_Small, Capacitor_SMD:C_0402_1005Metric_Pad0.74x0.62mm_HandSolder, F.Cu at (125.2, 121.0)
- added R5: R_Small, Capacitor_SMD:C_0402_1005Metric_Pad0.74x0.62mm_HandSolder, F.Cu at (132.5, 112.3)
- added R6: R_Small, Capacitor_SMD:C_0402_1005Metric_Pad0.74x0.62mm_HandSolder, F.Cu at (130.9, 115.6)
- added R7: 10k, Capacitor_SMD:C_0402_1005Metric_Pad0.74x0.62mm_HandSolder, F.Cu at (124.5, 119.0)
- added R8: 10k, Capacitor_SMD:C_0402_1005Metric_Pad0.74x0.62mm_HandSolder, F.Cu at (122.0, 122.9)
- added R9: 10k, Capacitor_SMD:C_0402_1005Metric_Pad0.74x0.62mm_HandSolder, F.Cu at (124.5, 117.0)
- added Y1: Crystal_GND3_Small, CSTCE8M00G55:OSC_CSTCE8M00G55-R0, F.Cu at (117.1, 125.8)
- U1: value STM32F103C8Tx -> MA730; footprint Package_QFP:LQFP-48_7x7mm_P0.5mm -> Package_DFN_QFN:QFN-16-1EP_3x3mm_P0.5mm_EP1.75x1.75mm; moved to B.Cu
- U4: value MA730 -> STM32F103C8T6; footprint Package_DFN_QFN:QFN-16-1EP_3x3mm_P0.5mm_EP1.75x1.75mm -> Package_QFP:LQFP-48_7x7mm_P0.5mm; moved to F.Cu
- moved U4 9.22 mm to (114.0, 115.0), turned to 0 degrees
- turned U1 to 180 degrees
Connections:
- J2 pad 3: unconnected-(J2-Pad3) -> USART2_RX
- J2 pad 4: unconnected-(J2-Pad4) -> USART2_TX
- J4 pad 1: unconnected-(J4-Pad1) -> +3V3
- J4 pad 2: unconnected-(J4-Pad2) -> GND
- J4 pad 3: unconnected-(J4-Pad3) -> SWCLK
- J4 pad 4: unconnected-(J4-Pad4) -> SWDIO
- U1 pad 10: unconnected-(U1-Pad10) -> GND
- U1 pad 12: unconnected-(U1-Pad12) -> SCK
- U1 pad 13: unconnected-(U1-Pad13) -> +3V3
- U1 pad 17: unconnected-(U1-Pad17) -> GND
- U1 pad 4: unconnected-(U1-Pad4) -> MOSI
- U1 pad 5: unconnected-(U1-Pad5) -> CS
- U1 pad 7: unconnected-(U1-Pad7) -> MISO
- U1 pad 8: unconnected-(U1-Pad8) -> GND
- U4 pad 1: unconnected-(U4-Pad1) -> +3V3
- U4 pad 10: unconnected-(U4-Pad10) -> EN1
- U4 pad 12: unconnected-(U4-Pad12) -> USART2_TX
- U4 pad 13: unconnected-(U4-Pad13) -> USART2_RX
- U4 pad 14: unconnected-(U4-Pad14) -> CS
- U4 pad 15: unconnected-(U4-Pad15) -> SCK
- U4 pad 16: unconnected-(U4-Pad16) -> MISO
- U4 pad 17: unconnected-(U4-Pad17) -> MOSI
- U4 pad 2: unconnected-(U4-Pad2) -> Net-(D1-Pad2)
- U4 pad 5: unconnected-(U4-Pad5) -> HSE_IN
- U4 pad 6: unconnected-(U4-Pad6) -> HSE_OUT
- U4 pad 7: unconnected-(U4-Pad7) -> Net-(C6-Pad1)
- U4 pad 8: unconnected-(U4-Pad8) -> GND
- U4 pad 9: unconnected-(U4-Pad9) -> +3V3

Commit message: update
Parts:
- added C24: 100nF, Capacitor_SMD:C_0402_1005Metric_Pad0.74x0.62mm_HandSolder, F.Cu at (163.0, 109.5)
- moved J1 0.25 mm to (124.0, 105.0)
Connections:
- C11 pad 1: unconnected-(C11-Pad1) -> +24V
- C11 pad 2: unconnected-(C11-Pad2) -> GND
- C12 pad 1: unconnected-(C12-Pad1) -> GND
- C12 pad 2: unconnected-(C12-Pad2) -> /VM
- C13 pad 1: unconnected-(C13-Pad1) -> Net-(R9-Pad1)
- C13 pad 2: unconnected-(C13-Pad2) -> GND
- C14 pad 1: unconnected-(C14-Pad1) -> Net-(C14-Pad1)
- C14 pad 2: unconnected-(C14-Pad2) -> GND
- C15 pad 1: unconnected-(C15-Pad1) -> Net-(U3-Pad1)
- C15 pad 2: unconnected-(C15-Pad2) -> Net-(U3-Pad6)
- C16 pad 1: unconnected-(C16-Pad1) -> +5V
- C16 pad 2: unconnected-(C16-Pad2) -> GND
- C17 pad 1: unconnected-(C17-Pad1) -> Net-(C17-Pad1)
- C17 pad 2: unconnected-(C17-Pad2) -> Net-(C17-Pad2)
- C18 pad 1: unconnected-(C18-Pad1) -> /VM
- C18 pad 2: unconnected-(C18-Pad2) -> Net-(U2-Pad3)
- C19 pad 1: unconnected-(C19-Pad1) -> /VM
- C19 pad 2: unconnected-(C19-Pad2) -> GND
- C20 pad 1: unconnected-(C20-Pad1) -> +5V
- C20 pad 2: unconnected-(C20-Pad2) -> GND
- C21 pad 1: unconnected-(C21-Pad1) -> +5V
- C21 pad 2: unconnected-(C21-Pad2) -> GND
- C22 pad 1: unconnected-(C22-Pad1) -> +3V3
- C22 pad 2: unconnected-(C22-Pad2) -> GND
- C23 pad 1: unconnected-(C23-Pad1) -> /VM
- C23 pad 2: unconnected-(C23-Pad2) -> GND
- J1 pad 1: unconnected-(J1-Pad1) -> +24V
- J1 pad 2: unconnected-(J1-Pad2) -> GND
- J1 pad 3: unconnected-(J1-Pad3) -> USART2_RX
- J1 pad 4: unconnected-(J1-Pad4) -> USART2_TX
- J2 pad 1: unconnected-(J2-Pad1) -> +24V
- J2 pad 2: unconnected-(J2-Pad2) -> GND
- J3 pad 1: unconnected-(J3-Pad1) -> +24V
- J3 pad 2: unconnected-(J3-Pad2) -> GND
- J3 pad 3: unconnected-(J3-Pad3) -> Step
- J3 pad 4: unconnected-(J3-Pad4) -> Dir
- R4 pad 1: unconnected-(R4-Pad1) -> +24V
- R4 pad 2: unconnected-(R4-Pad2) -> Net-(R4-Pad2)
- R5 pad 1: unconnected-(R5-Pad1) -> Net-(R5-Pad1)
- R5 pad 2: unconnected-(R5-Pad2) -> GND
- R6 pad 1: unconnected-(R6-Pad1) -> +5V
- R6 pad 2: unconnected-(R6-Pad2) -> Net-(R5-Pad1)
- R9 pad 1: unconnected-(R9-Pad1) -> Net-(R9-Pad1)
- R9 pad 2: unconnected-(R9-Pad2) -> +3V3
- U2 pad 1: unconnected-(U2-Pad1) -> Net-(C17-Pad1)
- U2 pad 10: unconnected-(U2-Pad10) -> BOUT1
- U2 pad 11: unconnected-(U2-Pad11) -> /VM
- U2 pad 12: unconnected-(U2-Pad12) -> Net-(C14-Pad1)
- U2 pad 13: unconnected-(U2-Pad13) -> Net-(C14-Pad1)
- U2 pad 14: unconnected-(U2-Pad14) -> GND
- U2 pad 15: unconnected-(U2-Pad15) -> Net-(C14-Pad1)
- U2 pad 16: unconnected-(U2-Pad16) -> Reset
- U2 pad 17: unconnected-(U2-Pad17) -> Net-(R9-Pad1)
- U2 pad 18: unconnected-(U2-Pad18) -> Net-(R9-Pad1)
- U2 pad 2: unconnected-(U2-Pad2) -> Net-(C17-Pad2)
- U2 pad 20: unconnected-(U2-Pad20) -> PWMB
- U2 pad 21: unconnected-(U2-Pad21) -> PWMA
- U2 pad 22: unconnected-(U2-Pad22) -> PWMC
- U2 pad 23: unconnected-(U2-Pad23) -> PWMD
- U2 pad 24: unconnected-(U2-Pad24) -> GND
- U2 pad 25: unconnected-(U2-Pad25) -> GND
- U2 pad 26: unconnected-(U2-Pad26) -> GND
- U2 pad 27: unconnected-(U2-Pad27) -> GND
- U2 pad 28: unconnected-(U2-Pad28) -> GND
- U2 pad 3: unconnected-(U2-Pad3) -> Net-(U2-Pad3)
- U2 pad 4: unconnected-(U2-Pad4) -> /VM
- U2 pad 5: unconnected-(U2-Pad5) -> AOUT1
- U2 pad 6: unconnected-(U2-Pad6) -> GND
- U2 pad 7: unconnected-(U2-Pad7) -> AOUT2
- U2 pad 8: unconnected-(U2-Pad8) -> BOUT2
- U2 pad 9: unconnected-(U2-Pad9) -> GND
- U3 pad 1: unconnected-(U3-Pad1) -> Net-(U3-Pad1)
- U3 pad 2: unconnected-(U3-Pad2) -> GND
- U3 pad 3: unconnected-(U3-Pad3) -> Net-(R5-Pad1)
- U3 pad 4: unconnected-(U3-Pad4) -> Net-(R4-Pad2)
- U3 pad 5: unconnected-(U3-Pad5) -> +24V
- U3 pad 6: unconnected-(U3-Pad6) -> Net-(U3-Pad6)
- U4 pad 10: EN1 -> Reset
- U4 pad 11: unconnected-(U4-Pad11) -> PWMD
- U5 pad 1: unconnected-(U5-Pad1) -> +5V
- U5 pad 2: unconnected-(U5-Pad2) -> GND
- U5 pad 3: unconnected-(U5-Pad3) -> +5V
- U5 pad 5: unconnected-(U5-Pad5) -> +3V3
