File: Stepper_Motor_FOC.kicad_sch (KiCad schematic)
At the start: 13 parts, among them J1 Conn_01x04, J2 Conn_01x04, J3 Conn_01x04, J4 Conn_01x04, U1 STM32F103C8Tx, U2 DRV8841, U3 ME3116, U4 MA730, U5 SPX3819M5-L-3-3

Commit message: update sch
Parts:
- removed U1: STM32F103C8Tx, Package_QFP:LQFP-48_7x7mm_P0.5mm, symbol MCU_ST_STM32F1:STM32F103C8Tx
- removed U4: MA730, Package_DFN_QFN:QFN-16-1EP_3x3mm_P0.5mm_EP1.75x1.75mm, symbol Sensor_Magnetic:MA730
- added C1, C4: 30PF, Capacitor_SMD:C_0402_1005Metric, symbol Device:C_Small
- added C10: 10uf, Capacitor_SMD:C_0402_1005Metric, symbol Device:C_Small
- added C12, C13, C14, C17, C18, C19: 100nF, Capacitor_SMD:C_0402_1005Metric_Pad0.74x0.62mm_HandSolder, symbol Device:C_Small
- added C15, C20: 4.7uF, Capacitor_SMD:C_0402_1005Metric_Pad0.74x0.62mm_HandSolder, symbol Device:C_Small
- added C16, C21, C22, C23: 47uF, Capacitor_SMD:C_1206_3216Metric_Pad1.33x1.80mm_HandSolder, symbol Device:C_Small
- added C2: 4u7, Capacitor_SMD:C_0402_1005Metric, symbol Device:C_Small
- added C3, C5, C6, C7, C8, C9: 100nf, Capacitor_SMD:C_0402_1005Metric, symbol Device:C_Small
- added D1: LED, LED_SMD:LED_0402_1005Metric, symbol Device:LED
- added JP1: SolderJumper_2_Open, Jumper:SoldJumper-2-P0.5mm_Open_RoundedPad, symbol Jumper:SolderJumper_2_Open
- added R1, R3: 10K, Resistor_SMD:R_0402_1005Metric, symbol Device:R_Small
- added R2: 1K5, Resistor_SMD:R_0402_1005Metric, symbol Device:R_Small
- added R4, R5: R_Small, Capacitor_SMD:C_0402_1005Metric_Pad0.74x0.62mm_HandSolder, symbol Device:R_Small
- added R7, R8, R9: 10k, Capacitor_SMD:C_0402_1005Metric_Pad0.74x0.62mm_HandSolder, symbol Device:R_Small
- added U1: MA730, Package_DFN_QFN:QFN-16-1EP_3x3mm_P0.5mm_EP1.75x1.75mm, symbol Sensor_Magnetic:MA730
- added U4: STM32F103C8T6, Package_QFP:LQFP-48_7x7mm_P0.5mm, symbol MCU_ST_STM32F1:STM32F103C8Tx
- added Y1: Crystal_GND3_Small, CSTCE8M00G55:OSC_CSTCE8M00G55-R0, symbol Device:Crystal_GND3_Small
- C11: renamed from C?; value C_Small -> 4.7uF; footprint (none) -> Capacitor_SMD:C_1206_3216Metric_Pad1.33x1.80mm_HandSolder
- R6: renamed from R?; footprint (none) -> Capacitor_SMD:C_0402_1005Metric_Pad0.74x0.62mm_HandSolder
- gave numbers to parts that had none: 2
Connections:
- net USART2_RX: now reaches J2.3 (Pin_3)
- net USART2_RX: now also U4.13 (PA3)
- net USART2_TX: now reaches J2.4 (Pin_4)
- net USART2_TX: now also U4.12 (PA2)
- net +3V3: now reaches J4.1 (Pin_1)
- net +3V3: now also C10.1, C2.1, C3.1, C5.1, C7.1, C8.1, C9.1, JP1.1 (A), R3.1, U1.13 (VDD), U4.1 (VBAT), U4.24 (VDD), U4.36 (VDD), U4.48 (VDD), U4.9 (VDDA)
- net GND: now reaches J4.2 (Pin_2)
- net GND: now also C1.2, C10.2, C2.2, C3.2, C4.2, C5.2, C6.2, C7.2, C8.2, C9.2, R1.2, R2.2, U1.10 (TEST), U1.17 (PAD), U1.8 (GND), U4.23 (VSS), U4.35 (VSS), U4.47 (VSS), U4.8 (VSSA), Y1.3
- net SWCLK: now reaches J4.3 (Pin_3)
- net SWCLK: now also U4.37 (PA14)
- net SWDIO: now reaches J4.4 (Pin_4)
- net SWDIO: now also U4.34 (PA13)
- new net: C6.1, R3.2, U4.7 (NRST)
- new net: D1.1 (K), R2.1
- new net: D1.2 (A), U4.2 (PC13)
- new net: JP1.2 (B), R1.1, U4.44 (BOOT0)
- new net Button: U4.18 (PB0)
- new net CS: U1.5 (~{CS}), U4.14 (PA4)
- new net EN1: U4.10 (PA0)
- new net ERROR: U4.22 (PB11)
- new net HSE_IN: C4.1, U4.5 (PD0), Y1.2
- new net HSE_OUT: C1.1, U4.6 (PD1), Y1.1
- new net I2C1_SCL: U4.42 (PB6)
- new net I2C1_SDA: U4.43 (PB7)
- new net MISO: U1.7 (MISO), U4.16 (PA6)
- new net MOSI: U1.4 (MOSI), U4.17 (PA7)
- new net PWMA: U4.29 (PA8)
- new net PWMB: U4.30 (PA9)
- new net PWMC: U4.31 (PA10)
- new net SCK: U1.12 (SCLK), U4.15 (PA5)
- new net SPI2_CS: U4.25 (PB12)
- new net SPI2_MISO: U4.27 (PB14)
- new net SPI2_MOSI: U4.28 (PB15)
- new net SPI2_SCK: U4.26 (PB13)
- new net USB_DM: U4.32 (PA11)
- new net USB_DP: U4.33 (PA12)
- no-connect marks 0 -> 21
Other:
- note added: "MA730"
- moved on the sheet: C11, D2, D3, J1, J2, J3, J4, U2, U3, U5

Commit message: update
Parts:
- removed R7, R8: 10k, Capacitor_SMD:C_0402_1005Metric_Pad0.74x0.62mm_HandSolder, symbol Device:R_Small
- added C24: 100nF, Capacitor_SMD:C_0402_1005Metric_Pad0.74x0.62mm_HandSolder, symbol Device:C_Small
- added L1: L_Small, Inductor_SMD:L_0420, symbol Device:L_Small
- D3: value D_Schottky_Small -> D
Connections:
- net EN1 is gone; now on net Reset: U4.10 (PA0)
- net +24V: now also C11.1, C19.1, C23.1, J1.1 (Pin_1), J2.1 (Pin_1), J3.1 (Pin_1), R4.1, U2.11 (VMB), U3.5 (Vin)
- net +3V3: now also C22.1, R9.2, U5.5 (OUT)
- net Dir: now also J3.4 (Pin_4)
- net GND: now also C11.2, C12.1, C13.2, C14.2, C16.2, C19.2, C20.2, C21.2, C22.2, C23.2, D3.2 (A), J1.2 (Pin_2), J2.2 (Pin_2), J3.2 (Pin_2), R5.2, U2.14 (GND), U2.24 (AI0), U2.25 (AI1), U2.26 (BI0), U2.27 (BI1), U2.28 (GND), U2.6 (AISEN), U2.9 (BISEN), U3.2 (GND), U5.2 (GND)
- net PWMA: now also U2.21 (AIN1)
- net PWMB: now also U2.20 (AIN2)
- net PWMC: now also U2.22 (BIN1)
- net Step: now also J3.3 (Pin_3)
- net USART2_RX: now also J1.3 (Pin_3)
- net USART2_TX: now also J1.4 (Pin_4)
- net at C14.1: now also U2.12 (AVREF), U2.13 (BVREF), U2.15 (V3P3OUT)
- net at R9.1: now also C13.1, U2.17 (nSlEEP), U2.18 (nfAULT)
- net PWMD: now reaches U4.11 (PA1)
- net PWMD: now also U2.23 (BIN2)
- net VM: now reaches C12.2
- net VM: now also C18.1, U2.4 (VMA)
- net at C15.1: now also U3.1 (BOOST)
- net at C15.2: now also D3.1 (K), U3.6 (SW), L1.1
- net +5V: now reaches U5.1 (IN)
- net +5V: now also C16.1, C20.1, C21.1, R6.1, U5.3 (EN), C24.1, L1.2
- net at R5.1: now also R6.2, U3.3 (Vfb), C24.2
- net at C17.1: now also U2.1 (CP1)
- net at C17.2: now also U2.2 (CP2)
- net at C18.2: now also U2.3 (VCP)
- net at R4.2: now also U3.4 (EN)
- net BOUT1: now reaches U2.10 (BOUT1)
- net Reset: now reaches U2.16 (NRESET)
- net AOUT1: now reaches U2.5 (AOUT1)
- net AOUT2: now reaches U2.7 (AOUT2)
- net BOUT2: now reaches U2.8 (BOUT2)
Other:
- moved on the sheet: C11, C12, C13, C14, C15, C16, C17, C18, C19, C20, C21, C22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
